File: DESIGN FILES/NANO-Minipops.kicad_pcb (KiCad board)
At the start: 2 copper layers, 68.6 x 53.3 mm, 21 parts, among them J1 Jack, J2 Conn_01x02, SW1 _, SW2 _, SW3 _, SW4 _, SW5 _, SW6 _, SW7 _, SW8 _

Commit message: Added BOM
Parts:
- C2: footprint Capacitors_THT:C_Rect_L7.0mm_W2.0mm_P5.00mm -> Resistors_Universal:Resistor_SMD+THTuniversal_0805to1206_RM10_HandSoldering
- moved C2 2.50 mm to (181.0, 51.0)
Routing:
- net GND: track 253.5 -> 256.1 mm
- net Net-(C1-Pad2): track 32.4 -> 35.0 mm
Changed lines of the file:
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@@
 (kicad_pcb (version 4) (host pcbnew 4.0.7)
   (general
-    (links 42)
+    (links 44)
     (no_connects 0)
     (area 146.924999 26.599999 215.650001 80.075001)
     (thickness 1.6)
     (drawings 20)
-    (tracks 182)
+    (tracks 184)
     (zones 0)
     (modules 21)
@@
     )
   )
-  (module Capacitors_THT:C_Rect_L7.0mm_W2.0mm_P5.00mm (layer F.Cu)
-    (at 183.5 51 180)
-    (descr "C, Rect series, Radial, pin pitch=5.00mm, , length*width=7*2mm^2, Capacitor")
-    (tags "C Rect series Radial pin pitch 5.00mm  length 7mm width 2mm Capacitor")
-    (fp_text reference C2 (at 2.5 -2.31 180) (layer F.SilkS)
-      (effects (font (size 1 1) (thickness 0.15)))
-    )
-    (fp_text value 100nF (at 2.5 2.31 180) (layer F.Fab)
-      (effects (font (size 1 1) (thickness 0.15)))
-    )
-    (fp_line (start -1 -1) (end -1 1) (layer F.Fab) (width 0.1))
-    (fp_line (start -1 1) (end 6 1) (layer F.Fab) (width 0.1))
-    (fp_line (start 6 1) (end 6 -1) (layer F.Fab) (width 0.1))
-    (fp_line (start 6 -1) (end -1 -1) (layer F.Fab) (width 0.1))
-    (fp_line (start -1.06 -1.06) (end 6.06 -1.06) (layer F.SilkS) (width 0.12))
-    (fp_line (start -1.06 1.06) (end 6.06 1.06) (layer F.SilkS) (width 0.12))
-    (fp_line (start -1.06 -1.06) (end -1.06 1.06) (layer F.SilkS) (width 0.12))
-    (fp_line (start 6.06 -1.06) (end 6.06 1.06) (layer F.SilkS) (width 0.12))
-    (fp_line (start -1.35 -1.35) (end -1.35 1.35) (layer F.CrtYd) (width 0.05))
-    (fp_line (start -1.35 1.35) (end 6.35 1.35) (layer F.CrtYd) (width 0.05))
-    (fp_line (start 6.35 1.35) (end 6.35 -1.35) (layer F.CrtYd) (width 0.05))
-    (fp_line (start 6.35 -1.35) (end -1.35 -1.35) (layer F.CrtYd) (width 0.05))
-    (fp_text user %R (at 2.5 0 180) (layer F.Fab)
-      (effects (font (size 1 1) (thickness 0.15)))
-    )
-    (pad 1 thru_hole circle (at 0 0 180) (size 1.6 1.6) (drill 0.8) (layers *.Cu *.Mask)
-      (net 2 "Net-(C1-Pad2)"))
-    (pad 2 thru_hole circle (at 5 0 180) (size 1.6 1.6) (drill 0.8) (layers *.Cu *.Mask)
-      (net 3 GND))
-    (model ${KISYS3DMOD}/Capacitors_THT.3dshapes/C_Rect_L7.0mm_W2.0mm_P5.00mm.wrl
-      (at (xyz 0 0 0))
-      (scale (xyz 1 1 1))
-      (rotate (xyz 0 0 0))
-    )
-  )
   (module LEDs:LED_D3.0mm (layer F.Cu)
     (at 151 31)
@@
       (xy 4.0005 1.524) (xy 4.098243 1.476146)) (layer B.SilkS) (width 0.01))
   )
+  (module Resistors_Universal:Resistor_SMD+THTuniversal_0805to1206_RM10_HandSoldering (layer F.Cu)
+    (at 181 51 180)
+    (descr "Resistor, SMD and THT, universal, 0805 to 1206,RM10,  Hand soldering,")
+    (tags "Resistor, SMD and THT, universal, 0805 to 1206, RM10, Hand soldering,")
+    (fp_text reference C2 (at 0 2.25 180) (layer F.SilkS)
+      (effects (font (size 1 1) (thickness 0.15)))
+    )
+    (fp_text value 100nF (at -0.39878 4.20116 180) (layer F.Fab)
+      (effects (font (size 1 1) (thickness 0.15)))
+    )
+    (fp_line (start 0 0.8001) (end 0.20066 0.8001) (layer F.SilkS) (width 0.15))
+    (fp_line (start 0 0.8001) (end -0.20066 0.8001) (layer F.SilkS) (width 0.15))
+    (fp_line (start -0.09906 -0.8001) (end -0.20066 -0.8001) (layer F.SilkS) (width 0.15))
+    (fp_line (start -0.20066 -0.8001) (end 0.20066 -0.8001) (layer F.SilkS) (width 0.15))
+    (pad 1 smd trapezoid (at -2.413 0 180) (size 3.50012 1.99898) (rect_delta 0.39878 0 ) (layers F.Cu F.Mask)
+      (net 2 "Net-(C1-Pad2)"))
+    (pad 2 smd trapezoid (at 2.413 0) (size 3.50012 1.99898) (rect_delta 0.39878 0 ) (layers F.Cu F.Mask)
+      (net 3 GND))
+    (pad 1 thru_hole rect (at -5.00126 0) (size 1.99898 1.99898) (drill 1.00076) (layers *.Cu *.Mask)
+      (net 2 "Net-(C1-Pad2)"))
+    (pad 2 thru_hole rect (at 5.00126 0) (size 1.99898 1.99898) (drill 1.00076) (layers *.Cu *.Mask)
+      (net 3 GND))
+  )
   (dimension 53.25 (width 0.3) (layer Eco1.User)
     (gr_text 53,250mm (at 221.85 53.375 90) (layer Eco1.User)
@@
   (segment (start 156.725 59.95) (end 151 54.225) (width 0.6) (layer F.Cu) (net 1))
   (segment (start 149.225 75.35) (end 156.725 67.85) (width 0.6) (layer F.Cu) (net 1))
+  (segment (start 183.413 51) (end 186.00126 51) (width 0.6) (layer F.Cu) (net 2) (status C00000))
   (segment (start 183.5 51) (end 182.85 51) (width 0.6) (layer F.Cu) (net 2))
   (segment (start 182.85 51) (end 179.925 53.925) (width 0.6) (layer F.Cu) (net 2))
@@
   (segment (start 164.087 51) (end 161.49874 51) (width 0.6) (layer F.Cu) (net 2))
   (segment (start 153.5 51) (end 161.49874 51) (width 0.6) (layer F.Cu) (net 2))
+  (segment (start 178.587 51) (end 175.99874 51) (width 1) (layer F.Cu) (net 3) (status C00000))
   (segment (start 200.50126 51) (end 205.825 51) (width 1) (layer F.Cu) (net 3))
   (segment (start 205.825 51) (end 207.825 49) (width 1) (layer F.Cu) (net 3))
@@
   (segment (start 190.675 66.675) (end 193 69) (width 1) (layer F.Cu) (net 3))
   (segment (start 190.49874 51) (end 188.8 51) (width 0.6) (layer F.Cu) (net 4))
+  (segment (start 188.8 51) (end 185.7 47.9) (width 0.6) (layer F.Cu) (net 4))
   (segment (start 148.3 33.7) (end 151 31) (width 0.6) (layer B.Cu) (net 4))
   (segment (start 148.3 46.1) (end 148.3 33.7) (width 0.6) (layer B.Cu) (net 4))
@@
   (segment (start 185.7 47.9) (end 185.6 47.8) (width 0.6) (layer B.Cu) (net 4))
   (via (at 185.7 47.9) (size 0.6) (drill 0.4) (layers F.Cu B.Cu) (net 4))
-  (segment (start 188.8 51) (end 185.7 47.9) (width 0.6) (layer F.Cu) (net 4))
   (segment (start 193.087 51) (end 190.49874 51) (width 0.6) (layer F.Cu) (net 4))
   (segment (start 149 56) (end 149 35.6) (width 0.6) (layer F.Cu) (net 5))
